Commit message: update
update

File: ssctractor/urdf/tractor_notgazebo.urdf (robot description, URDF)
Before this commit: robot tractor, 7 links, 6 joints
Links:
- removed link robot_footprint
- added link base_footprint
- link base_link: mass 15.0 -> 30.0; geometry collision box size=.65 .4 .2; collision sphere radius=0.0375
- link left_wheel: mass 5.0 -> 3.0
- link right_wheel: mass 5.0 -> 3.0
Joints:
- removed joint robot_footprint_joint
- added joint base_link_joint: type fixed, parent base_footprint, child base_link, origin xyz=0 0 0.1 rpy=0 0 0
- joint camera_joint: origin xyz=0.3 0 0.18 rpy=0 0 0 -> xyz=0.0 0 0.1 rpy=0 -1.5705 0
- joint imu_joint: origin xyz=0 0 .2 rpy=0 0 0 -> xyz=-0.0205 0 0.251 rpy=0 0 0
- joint laser_joint: origin xyz=0.3 0.0 0.13 rpy=0 0 0 -> xyz=0.08 0.0 0.3 rpy=0 0 3.14159265

Commit message: navigation update
11/03

File: ssctractor/urdf/tractor_notgazebo.urdf (robot description, URDF)
Before this commit: robot tractor, 7 links, 6 joints
Joints:
- joint camera_joint: origin xyz=0.0 0 0.1 rpy=0 -1.5705 0 -> xyz=0.0 0 0.1 rpy=0 0 3.141592
