Commit message: update lino
update_lino

File: linorobot2_description/urdf/2wd_properties.urdf.xacro (robot description, xacro)
@@ -8,5 +8,5 @@
   <xacro:property name="trailer_width" value="0.6" />
   <xacro:property name="trailer_height" value="0.2" />
-  <xacro:property name="trailer_mass" value="27" />
+  <xacro:property name="trailer_mass" value="50" />
 <!--  <xacro:property name="base_length1" value="0.492" />
   <xacro:property name="base_width1" value="0.447" />
